File: YY1705K1A0_breakout.kicad_sch (KiCad schematic)
At the start: 7 parts, among them J1 ESP32_HDR_7, J2 FPC_ZIF_12_0.5mm

Commit message: Convert SMD passives to through-hole (THT)
Replace all five 0402 SMD passive components with through-hole
equivalents. Board dimensions (34x53mm) and single-layer F.Cu
constraint are preserved. J2 FPC ZIF connector remains SMD.

Component changes:
- R1 22R : SMD 0402 -> axial DIN0207 7.62mm pitch horizontal
- R2 10k : SMD 0402 -> axial DIN0207 5.08mm pitch vertical mount
- R3 10k : SMD 0402 -> axial DIN0207 5.08mm pitch vertical mount
- C1 10uF: SMD 0402 -> ceramic disc / radial THT 5mm pitch
- C2 100nF: SMD 0402 -> ceramic disc THT 5mm pitch

PCB layout:
- R2/R3 placed at Y=8.5 (just below J1) with pads landing
  directly on the RESET and CS signal traces, minimising extra routing
- C1/C2 moved to right clear-zone (X=26-32) where no signal
  diagonals pass
- R1 +3V3 routed via bottom loop (Y=51) to avoid crossing the
  five signal diagonal traces
- All routing remains single-layer F.Cu only

Files changed: kicad_pcb, kicad_sch, BOM.csv, README.md
Parts:
- C1, C2: footprint Capacitor_SMD:C_0402_1005Metric -> Capacitor_THT:C_Disc_D5.0mm_W2.5mm_P5.00mm
- R1: footprint Resistor_SMD:R_0402_1005Metric -> Resistor_THT:R_Axial_DIN0207_L6.3mm_D2.5mm_P7.62mm_Horizontal
- R2, R3: footprint Resistor_SMD:R_0402_1005Metric -> Resistor_THT:R_Axial_DIN0207_L6.3mm_D2.5mm_P5.08mm_Vertical
Changed lines of the file:
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@@
     (property "Reference" "R1" (id 0) (at 140.0 27.3 0) (effects (font (size 1.27 1.27))))
     (property "Value" "22R" (id 1) (at 140.0 29.84 0) (effects (font (size 1.27 1.27))))
-    (property "Footprint" "Resistor_SMD:R_0402_1005Metric" (id 2) (at 140.0 40.0 0) (effects (font (size 1.27 1.27)) hide))
+    (property "Footprint" "Resistor_THT:R_Axial_DIN0207_L6.3mm_D2.5mm_P7.62mm_Horizontal" (id 2) (at 140.0 40.0 0) (effects (font (size 1.27 1.27)) hide))
     (property "Datasheet" "" (id 3) (at 140.0 40.0 0) (effects (font (size 1.27 1.27)) hide))
     (pin "1")
@@
     (property "Reference" "R2" (id 0) (at 140.0 47.3 0) (effects (font (size 1.27 1.27))))
     (property "Value" "10k" (id 1) (at 140.0 49.84 0) (effects (font (size 1.27 1.27))))
-    (property "Footprint" "Resistor_SMD:R_0402_1005Metric" (id 2) (at 140.0 60.0 0) (effects (font (size 1.27 1.27)) hide))
+    (property "Footprint" "Resistor_THT:R_Axial_DIN0207_L6.3mm_D2.5mm_P5.08mm_Vertical" (id 2) (at 140.0 60.0 0) (effects (font (size 1.27 1.27)) hide))
     (property "Datasheet" "" (id 3) (at 140.0 60.0 0) (effects (font (size 1.27 1.27)) hide))
     (pin "1")
@@
     (property "Reference" "R3" (id 0) (at 140.0 67.3 0) (effects (font (size 1.27 1.27))))
     (property "Value" "10k" (id 1) (at 140.0 69.84 0) (effects (font (size 1.27 1.27))))
-    (property "Footprint" "Resistor_SMD:R_0402_1005Metric" (id 2) (at 140.0 80.0 0) (effects (font (size 1.27 1.27)) hide))
+    (property "Footprint" "Resistor_THT:R_Axial_DIN0207_L6.3mm_D2.5mm_P5.08mm_Vertical" (id 2) (at 140.0 80.0 0) (effects (font (size 1.27 1.27)) hide))
     (property "Datasheet" "" (id 3) (at 140.0 80.0 0) (effects (font (size 1.27 1.27)) hide))
     (pin "1")
@@
     (property "Reference" "C1" (id 0) (at 140.0 92.3 0) (effects (font (size 1.27 1.27))))
     (property "Value" "10uF" (id 1) (at 140.0 94.84 0) (effects (font (size 1.27 1.27))))
-    (property "Footprint" "Capacitor_SMD:C_0402_1005Metric" (id 2) (at 140.0 105.0 0) (effects (font (size 1.27 1.27)) hide))
+    (property "Footprint" "Capacitor_THT:C_Disc_D5.0mm_W2.5mm_P5.00mm" (id 2) (at 140.0 105.0 0) (effects (font (size 1.27 1.27)) hide))
     (property "Datasheet" "" (id 3) (at 140.0 105.0 0) (effects (font (size 1.27 1.27)) hide))
     (pin "1")
@@
     (property "Reference" "C2" (id 0) (at 160.0 92.3 0) (effects (font (size 1.27 1.27))))
     (property "Value" "100nF" (id 1) (at 160.0 94.84 0) (effects (font (size 1.27 1.27))))
-    (property "Footprint" "Capacitor_SMD:C_0402_1005Metric" (id 2) (at 160.0 105.0 0) (effects (font (size 1.27 1.27)) hide))
+    (property "Footprint" "Capacitor_THT:C_Disc_D5.0mm_W2.5mm_P5.00mm" (id 2) (at 160.0 105.0 0) (effects (font (size 1.27 1.27)) hide))
     (property "Datasheet" "" (id 3) (at 160.0 105.0 0) (effects (font (size 1.27 1.27)) hide))
     (pin "1")
@@
   (symbol_instances
     (path "/fda0368a-167f-4599-a5ea-1e36e8848717" (reference "J1") (unit 1) (value "ESP32_HDR_7") (footprint "Connector_PinHeader_2.54mm:PinHeader_1x07_P2.54mm_Vertical"))
-    (path "/389a5d39-0236-4bac-8132-0a354aa23aa9" (reference "R1") (unit 1) (value "22R") (footprint "Resistor_SMD:R_0402_1005Metric"))
-    (path "/114a434d-0cbb-4b99-90e0-6179532c7905" (reference "R2") (unit 1) (value "10k") (footprint "Resistor_SMD:R_0402_1005Metric"))
-    (path "/b4694948-f34c-42e8-afaf-7ff368040334" (reference "R3") (unit 1) (value "10k") (footprint "Resistor_SMD:R_0402_1005Metric"))
-    (path "/86b814ae-d688-4cfa-9a3c-72b36d777748" (reference "C1") (unit 1) (value "10uF") (footprint "Capacitor_SMD:C_0402_1005Metric"))
-    (path "/0a03aced-67cf-4f8f-bd7d-5eefca690abe" (reference "C2") (unit 1) (value "100nF") (footprint "Capacitor_SMD:C_0402_1005Metric"))
+    (path "/389a5d39-0236-4bac-8132-0a354aa23aa9" (reference "R1") (unit 1) (value "22R") (footprint "Resistor_THT:R_Axial_DIN0207_L6.3mm_D2.5mm_P7.62mm_Horizontal"))
+    (path "/114a434d-0cbb-4b99-90e0-6179532c7905" (reference "R2") (unit 1) (value "10k") (footprint "Resistor_THT:R_Axial_DIN0207_L6.3mm_D2.5mm_P5.08mm_Vertical"))
+    (path "/b4694948-f34c-42e8-afaf-7ff368040334" (reference "R3") (unit 1) (value "10k") (footprint "Resistor_THT:R_Axial_DIN0207_L6.3mm_D2.5mm_P5.08mm_Vertical"))
+    (path "/86b814ae-d688-4cfa-9a3c-72b36d777748" (reference "C1") (unit 1) (value "10uF") (footprint "Capacitor_THT:C_Disc_D5.0mm_W2.5mm_P5.00mm"))
+    (path "/0a03aced-67cf-4f8f-bd7d-5eefca690abe" (reference "C2") (unit 1) (value "100nF") (footprint "Capacitor_THT:C_Disc_D5.0mm_W2.5mm_P5.00mm"))
     (path "/745b2f1b-07de-48f8-a038-a1e2156cf615" (reference "J2") (unit 1) (value "FPC_ZIF_12_0.5mm") (footprint "Local:FPC_12_0.5mm"))
   )
